Commit message: Fix aruco_moveit_config gripper mismatch and initial_positions xacro arg collisions
Regenerated aruco_moveit_config from ur.urdf.xacro (RG2 gripper) to
match the actual Gazebo sim robot, replacing the stale Robotiq-85-based
config that caused "joint not found" errors in move_group/RViz.

Renamed the package's initial_positions_file xacro:arg to
ros2_control_initial_positions_file to stop it colliding with
ur.urdf.xacro's identically-named arg — xacro args share one global
namespace, so the collision silently fed the wrong (wrong-shaped)
YAML into ros2_control's initial_positions lookup.

File: aruco_moveit_config/config/name.ros2_control.xacro (robot description, xacro)
@@ -2,5 +2,5 @@
 <robot xmlns:xacro="http://www.ros.org/wiki/xacro">
     <xacro:macro name="name_ros2_control" params="name initial_positions_file">
-        <xacro:property name="initial_positions" value="${load_yaml(initial_positions_file)['initial_positions']}"/>
+        <xacro:property name="initial_positions" value="${xacro.load_yaml(initial_positions_file)['initial_positions']}"/>
         <ros2_control name="${name}" type="system">
             <hardware>

File: aruco_moveit_config/config/name.urdf.xacro (robot description, xacro)
@@ -1,9 +1,9 @@
 <?xml version="1.0"?>
 <robot xmlns:xacro="http://www.ros.org/wiki/xacro" name="name">
-    <xacro:arg name="initial_positions_file" default="initial_positions.yaml" />
+    <xacro:arg name="ros2_control_initial_positions_file" default="$(find aruco_moveit_config)/config/initial_positions.yaml" />
     <!-- Import name urdf file -->
     <xacro:include filename="$(find ur_description)/urdf/ur.urdf.xacro" />
     <!-- Import control_xacro -->
     <xacro:include filename="name.ros2_control.xacro" />
-    <xacro:name_ros2_control name="FakeSystem" initial_positions_file="$(arg initial_positions_file)"/>
+    <xacro:name_ros2_control name="FakeSystem" initial_positions_file="$(arg ros2_control_initial_positions_file)"/>
 </robot>
